Commit message: Updated urdf file

File: urdf/arm.urdf (robot description, URDF)
Before this commit: robot arm, 7 links, 6 joints
Joints:
- joint base_to_link1: axis (none) -> 0 0 1; limit (none) -> lower=-3.14 upper=3.14 effort=0.0 velocity=0.0; type fixed -> revolute
- joint link1_to_link2: axis (none) -> 0.0 0.0 1.0; limit (none) -> lower=-1.57 upper=1.57 effort=0.0 velocity=0.0; origin xyz=0.0 0.0 0.0 rpy=0.0 0.0 5 -> xyz=0.0 0.0 0.0 rpy=0.0 -1.56 -1.58; type fixed -> revolute
- joint link2_to_link3: axis (none) -> 0.0 0.0 1; limit (none) -> lower=-0.0 upper=3.14 effort=0.0 velocity=0.0; origin xyz=0.0 0.0 0.0 rpy=0.0 0.0 0.0 -> xyz=0.2 0.0 0.0 rpy=3.15 0.0 1.57; type fixed -> revolute
- joint link3_to_link4: axis (none) -> 0.0 0.0 1.0; limit (none) -> lower=0 upper=3.14 effort=0.0 velocity=0.0; origin xyz=0.0 0.0 0.0 rpy=0.0 0.0 0.0 -> xyz=0.087 -0.225 0.0 rpy=1.55 0.0 0.0; type fixed -> revolute
- joint link4_to_link5: axis (none) -> 0.0 1.0 0.0; limit (none) -> lower=-3.14 upper=1.57 effort=0.0 velocity=0.0; origin xyz=0.0 0.0 0.0 rpy=0.0 0.0 0.0 -> xyz=0.0 0.0 0.0 rpy=3.15 3.16 0; type fixed -> revolute
- joint link5_to_link6: origin xyz=0.0 0.0 0.0 rpy=0.0 0.0 0.0 -> xyz=0.0 0.0 0.06 rpy=0.0 0.0 3.1
